File: iris_microphone_only/iris_microphone_only.kicad_sch (KiCad schematic)
At the start: 0 parts

Commit message: redesigned notch filter for microphone
Parts:
- added C1, C14, C18, C19: 0.1u, symbol Device:C_Small
- added C17: 0.2u, symbol Device:C_Small
- added R1, R30: 26.7K, symbol Device:R_US
- added R18: 22K, symbol Device:R_US
- added R19: 820K, symbol Device:R_US
- added R27: 13K, symbol Device:R_US
- added R32: 6.2K, symbol Device:R_US
- added U2: ${SIM.PARAMS}, symbol Simulation_SPICE:OPAMP
- added V1: 3.3, symbol Simulation_SPICE:VDC
- added V2: VSIN, symbol Simulation_SPICE:VSIN
- added V3: VPWL, symbol Simulation_SPICE:VPWL
Connections:
- new net: C1.2, C18.1, R27.1
- new net: C17.1, R1.2, R30.1
- new net: R18.1, R19.2, U2.2 (-)
- new net +3V3: C14.1, U2.3 (V+), V1.1
- new net ENV_OUT: R19.1, U2.5
- new net GND: C14.2, C17.2, C19.2, R18.2, R27.2, U2.4 (V-), V1.2, V2.2, V3.2
- new net LPF: C18.2, C19.1, R30.2, R32.1
- new net PWL: R32.2, V2.1
- new net notch: C1.1, R1.1, U2.1 (+)
